File: Schematics/esp07.sch (EAGLE design)
At the start: 5 parts

Commit message: as
Parts:
- removed C1: 104, adafruit:C-USC0805
- removed R1: 10k, adafruit:R-US_M0805
- removed X1, X2: (no value), adafruit:ESP-12
- added C2: (no value), SparkFun-Capacitors:CAP0805
- added R2: (no value), SparkFun-Resistors:RESISTOR0805-RES
- added U$1: ESP8266-03, lio:ESP8266-03
Changed lines of the file:
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@@
 <layer number="56" name="wert" color="7" fill="1" visible="no" active="no"/>
 <layer number="57" name="tCAD" color="7" fill="1" visible="no" active="no"/>
+<layer number="59" name="tCarbon" color="7" fill="1" visible="no" active="no"/>
+<layer number="60" name="bCarbon" color="7" fill="1" visible="no" active="no"/>
 <layer number="90" name="Modules" color="5" fill="1" visible="yes" active="yes"/>
 <layer number="91" name="Nets" color="2" fill="1" visible="yes" active="yes"/>
@@
 <layer number="127" name="_tValues" color="7" fill="1" visible="no" active="yes"/>
 <layer number="128" name="_bValues" color="7" fill="1" visible="no" active="yes"/>
+<layer number="129" name="Mask" color="7" fill="1" visible="yes" active="yes"/>
 <layer number="131" name="tAdjust" color="7" fill="1" visible="no" active="yes"/>
 <layer number="132" name="bAdjust" color="7" fill="1" visible="no" active="yes"/>
@@
 <layer number="223" name="223bmp" color="24" fill="1" visible="no" active="no"/>
 <layer number="224" name="224bmp" color="25" fill="1" visible="no" active="no"/>
+<layer number="225" name="225bmp" color="7" fill="1" visible="yes" active="yes"/>
+<layer number="226" name="226bmp" color="7" fill="1" visible="yes" active="yes"/>
+<layer number="227" name="227bmp" color="7" fill="1" visible="yes" active="yes"/>
+<layer number="228" name="228bmp" color="7" fill="1" visible="yes" active="yes"/>
+<layer number="229" name="229bmp" color="7" fill="1" visible="yes" active="yes"/>
+<layer number="230" name="230bmp" color="7" fill="1" visible="yes" active="yes"/>
 <layer number="231" name="Eagle3D_PG1" color="7" fill="1" visible="no" active="no"/>
 <layer number="232" name="Eagle3D_PG2" color="7" fill="1" visible="no" active="no"/>
@@
 <layer number="251" name="SMDround" color="7" fill="1" visible="no" active="no"/>
 <layer number="254" name="cooling" color="7" fill="1" visible="no" active="yes"/>
+<layer number="255" name="routoute" color="7" fill="1" visible="yes" active="yes"/>
 </layers>
 <schematic xreflabel="%F%N/%S.%C%R" xrefpart="/%S.%C%R">
@@
 </classes>
 <parts>
-<part name="X1" library="adafruit" deviceset="ESP-12" device=""/>
-<part name="X2" library="adafruit" deviceset="ESP-12" device=""/>
 <part name="CN1" library="adafruit" deviceset="USB" device="MOLEX"/>
-<part name="R1" library="adafruit" deviceset="R-US_" device="M0805" value="10k"/>
-<part name="C1" library="adafruit" deviceset="C-US" device="C0805" value="104"/>
+<part name="C2" library="SparkFun-Capacitors" deviceset="CAP" device="0805"/>
+<part name="R2" library="SparkFun-Resistors" deviceset="RESISTOR" device="0805-RES"/>
+<part name="U$1" library="lio" deviceset="ESP8266-03" device=""/>
 </parts>
 <sheets>
@@
 </plain>
 <instances>
-<instance part="X1" gate="G$1" x="27.94" y="71.12"/>
-<instance part="X2" gate="G$1" x="68.58" y="71.12"/>
 <instance part="CN1" gate="G$1" x="25.4" y="104.14"/>
-<instance part="R1" gate="G$1" x="53.34" y="104.14"/>
-<instance part="C1" gate="G$1" x="40.64" y="119.38"/>
+<instance part="C2" gate="G$1" x="40.64" y="99.06"/>
+<instance part="R2" gate="G$1" x="53.34" y="93.98"/>
+<instance part="U$1" gate="G$1" x="76.2" y="116.84"/>
 </instances>
 <busses>
